File: rufous/rufous_choc_hybrid.kicad_pcb (KiCad board)
At the start: 2 copper layers, 209.8 x 99 mm, 35 parts

Commit message: Update kicad files
Connections:
- S29 pad 1: P5 -> P4
Routing:
- net P4: track 228.4 -> 267.2 mm, vias 4 -> 5
- net P10: track 218.9 -> 236.2 mm
- net P5: track 291.1 -> 288.9 mm
