File: rufous/rufous_mx.kicad_pcb (KiCad board)
At the start: 2 copper layers, 215.3 x 102.8 mm, 35 parts

Commit message: Update kicad files
Connections:
- S29 pad 1: P5 -> P4
Routing:
- net P4: track 189.1 -> 217.0 mm, vias 4 -> 5
- net P5: track 234.2 -> 223.2 mm
